File: UccMicroDuino/2610946-Dante-Franco-Microduino/2610946-Dante-Franco-Microduino.kicad_pcb (KiCad board)
At the start: 2 copper layers, 8 parts, among them J1 Conn_01x10_Socket, J2 USB_A, U1 ATtiny85-20S

Commit message: Entrega Placa
Parts:
- added D4: Led Green, ledSmd:ledSMD, F.Cu at (180.0, 87.0)
- added D5: LED, ledSmd:ledSMD, F.Cu at (206.5, 74.0)
- added R2: 68Ω 5% 1/8W, Resistor_SMD:R_0805_2012Metric_Pad1.20x1.40mm_HandSolder, F.Cu at (177.5, 77.5)
- added R3: 68Ω 5% 1/8W, Resistor_SMD:R_0805_2012Metric_Pad1.20x1.40mm_HandSolder, F.Cu at (187.5, 77.0)
- added R4: 330Ω 5% 1/8W, Resistor_SMD:R_0805_2012Metric_Pad1.20x1.40mm_HandSolder, F.Cu at (183.0, 92.5)
- added R5: 330Ω 5% 1/8W, Resistor_SMD:R_0805_2012Metric_Pad1.20x1.40mm_HandSolder, F.Cu at (193.5, 72.5)
- C1: value C -> 0.1u
- D1: value D_Filled -> PMLL4148L
- D2: value D_Zener -> 3.6V 1/2mW
- D3: value LED -> 3.6V 1/2mW; footprint ledSmd:ledSMD -> Diode_SMD:D_SOD-123
- J1: value Conn_01x10_Socket -> Pcb USB Type A; footprint Connector_PinHeader_2.54mm:PinHeader_1x10_P2.54mm_Vertical -> embeddedPcbUsb:USB_A_UCC
- J2: value USB_A -> Header; footprint embeddedPcbUsb:USB_A_UCC -> Connector_PinHeader_2.54mm:PinHeader_1x10_P2.54mm_Vertical
- R1: value R -> 1.5KΩ 5% 1/8W
- U1: value ATtiny85-20S -> ATtiny85-20SU
- moved C1 73.3 mm to (210.0, 84.0), turned to 180 degrees
- moved U1 61.8 mm to (193.3, 86.9), turned to 180 degrees
- moved J2 55.4 mm to (180.7, 98.5), turned to 90 degrees
- moved D2 52.2 mm to (178.0, 71.8), turned to 90 degrees
- moved J1 51.0 mm to (175.0, 64.7), turned to -90 degrees
- moved D3 47.8 mm to (181.5, 74.2), turned to 90 degrees
- moved D1 44.3 mm to (171.5, 72.8), turned to 90 degrees
- moved R1 35.2 mm to (173.0, 77.5)
Connections:
- C1 pad 1: unconnected-(C1-Pad1) -> +5V
- C1 pad 2: unconnected-(C1-Pad2) -> GND
- D1 pad 2: unconnected-(D1-A-Pad2) -> Net-(D1-A)
- D2 pad 1: unconnected-(D2-K-Pad1) -> Net-(D2-K)
- D2 pad 2: unconnected-(D2-A-Pad2) -> GND
- D3 pad 1: unconnected-(D3-K-Pad1) -> Net-(D3-K)
- D3 pad 2: unconnected-(D3-A-Pad2) -> GND
- J1 pad 1: unconnected-(J1-Pin_1-Pad1) -> Net-(D1-A)
- J1 pad 2: unconnected-(J1-Pin_2-Pad2) -> Net-(D2-K)
- J1 pad 3: unconnected-(J1-Pin_3-Pad3) -> Net-(D3-K)
- J1 pad 4: unconnected-(J1-Pin_4-Pad4) -> GND
- J2 pad 1: unconnected-(J2-VBUS-Pad1) -> +5V
- J2 pad 2: unconnected-(J2-D--Pad2) -> GND
- J2 pad 4: unconnected-(J2-GND-Pad4) -> Net-(J2-Pin_4)
- R1 pad 2: unconnected-(R1-Pad2) -> Net-(D2-K)
- U1 pad 1: unconnected-(U1-~{RESET}/PB5-Pad1) -> Net-(J2-Pin_9)
- U1 pad 2: unconnected-(U1-XTAL1/PB3-Pad2) -> Net-(J2-Pin_7)
- U1 pad 3: unconnected-(U1-XTAL2/PB4-Pad3) -> Net-(J2-Pin_8)
- U1 pad 4: unconnected-(U1-GND-Pad4) -> GND
- U1 pad 5: unconnected-(U1-AREF/PB0-Pad5) -> Net-(J2-Pin_4)
- U1 pad 6: unconnected-(U1-PB1-Pad6) -> Net-(D4-A)
- U1 pad 7: unconnected-(U1-PB2-Pad7) -> Net-(J2-Pin_6)
- U1 pad 8: unconnected-(U1-VCC-Pad8) -> +5V
Routing:
- net +5V: track 0.00 -> 118.7 mm
- net GND: track 0.00 -> 97.4 mm
- net Net-(J2-Pin_8): track 0.00 -> 42.2 mm
- net Net-(J2-Pin_7): track 0.00 -> 38.8 mm
- net Net-(D4-A): track 0.00 -> 32.7 mm
- net Net-(D3-K): track 0.00 -> 19.9 mm
- net Net-(D2-K): track 0.00 -> 19.6 mm
- net Net-(J2-Pin_4): track 0.00 -> 17.4 mm
- net Net-(J2-Pin_6): track 0.00 -> 14.9 mm
- net Net-(J2-Pin_9): track 0.00 -> 11.4 mm
- net Net-(D5-K): track 0.00 -> 10.8 mm
- net Net-(D1-A): track 0.00 -> 6.50 mm
- net Net-(D4-K): track 0.00 -> 4.40 mm
Other:
- board outline added: 45 x 45 mm
