File: UccMicroDuino/2610946-Dante-Franco-Microduino/2610946-Dante-Franco-Microduino.kicad_sch (KiCad schematic)
At the start: 14 parts, among them J1 Pcb USB Type A, J2 Header, U1 ATtiny85-20SU

Commit message: Entrega Placa
Parts:
- D3: footprint (none) -> Diode_SMD:D_SOD-123
- R2, R3, R4, R5: footprint (none) -> Resistor_SMD:R_0805_2012Metric_Pad1.20x1.40mm_HandSolder
- renumbered D3 to D5
Changed lines of the file:
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@@
-	)
-	(junction
-		(at 147.32 72.39)
-		(diameter 0)
-		(color 0 0 0 0)
 	)
 	(junction
@@
 	(wire
 		(pts
-			(xy 147.32 72.39) (xy 147.32 73.66)
-		)
-		(stroke
-			(width 0)
-			(type default)
-		)
-	)
-	(wire
-		(pts
 			(xy 173.99 100.33) (xy 173.99 105.41)
 		)
@@
 	(wire
 		(pts
+			(xy 82.55 121.92) (xy 82.55 125.73)
+		)
+		(stroke
+			(width 0)
+			(type default)
+		)
+	)
+	(wire
+		(pts
 			(xy 147.32 67.31) (xy 147.32 72.39)
-		)
-		(stroke
-			(width 0)
-			(type default)
-		)
-	)
-	(wire
-		(pts
-			(xy 82.55 121.92) (xy 82.55 125.73)
 		)
 		(stroke
@@
 		(dnp no)
 		(fields_autoplaced yes)
-		(property "Reference" "D3"
+		(property "Reference" "D5"
 			(at 259.08 75.2474 90)
 			(show_name no)
@@
 			(project "2610946-Dante-Franco-Microduino"
 				(path "/f2c20679-f28d-47ad-9191-2bfbde129570"
-					(reference "D3")
+					(reference "D5")
 					(unit 1)
 				)
@@
 			)
 		)
-		(property "Footprint" ""
+		(property "Footprint" "Resistor_SMD:R_0805_2012Metric_Pad1.20x1.40mm_HandSolder"
 			(at 109.22 102.362 90)
 			(hide yes)
@@
 		)
 		(property "Value" "330Ω  5% 1/8W"
-			(at 173.228 67.31 90)
-			(show_name no)
-			(do_not_autoplace no)
-			(effects
-				(font
-					(size 1.27 1.27)
-				)
-			)
-		)
-		(property "Footprint" ""
+			(at 172.974 66.04 90)
+			(show_name no)
+			(do_not_autoplace no)
+			(effects
+				(font
+					(size 1.27 1.27)
+				)
+			)
+		)
+		(property "Footprint" "Resistor_SMD:R_0805_2012Metric_Pad1.20x1.40mm_HandSolder"
 			(at 172.72 71.628 90)
 			(hide yes)
@@
 			)
 		)
-		(property "Footprint" ""
+		(property "Footprint" "Resistor_SMD:R_0805_2012Metric_Pad1.20x1.40mm_HandSolder"
 			(at 99.06 103.378 90)
 			(hide yes)
@@
 			)
 		)
-		(property "Footprint" ""
+		(property "Footprint" "Diode_SMD:D_SOD-123"
 			(at 90.17 114.3 0)
 			(hide yes)
@@
 			)
 		)
-		(property "Footprint" ""
+		(property "Footprint" "Resistor_SMD:R_0805_2012Metric_Pad1.20x1.40mm_HandSolder"
 			(at 253.492 87.63 90)
 			(hide yes)
